File: Multiplatine.kicad_pcb (KiCad board)
At the start: 2 copper layers, 100 x 100 mm, 64 parts, among them J1 Pogo Pins (QWIIC), J10 Conn_01x02_Male, J12 Conn_02x03_Odd_Even, J13 Conn_02x03_Odd_Even, J14 USB_B_Micro, J2 AUDIO Left, J3 AUDIO Right, J4 SD Card, J5 Flo Display, J6 Brightness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

Commit message: Initial commit
Parts:
- added S2: JS5208, digikey-footprints:Switch_Nav_12.4x12.4mm_SMD_JS5208, F.Cu at (85.0, 119.5)
- added S3: NAV_SWITCH, Switches:NAV_SWITCH, F.Cu at (40.6, 83.8)
Other:
- net class Default removed
