File: Multiplatine.kicad_sch (KiCad schematic)
At the start: 1 part, among them U1 ESP32-S2-WROVER

Commit message: Initial commit
Parts:
- removed U1: ESP32-S2-WROVER, RF_Module:ESP32-S2-WROVER, symbol RF_Module:ESP32-S2-WROVER
- added BT1: (no value), symbol Device:Battery_Cell
- added C1, C10, C11, C12, C13, C14, C15, C16, C17, C2, C3, C4, C5, C6, C7, C8, C9: (no value), symbol Device:C_Small
- added D1: (no value), symbol Device:LED_Small
- added D2, D3, D4: (no value), symbol LED:WS2812B
- added D5: (no value), symbol Device:D_Schottky
- added DS1: (no value), symbol Multiplatine-rescue:SLP3-200-100-F-SLP3-200-100-F_Lightpipe
- added FB1, FB2, FB3, FB4: (no value), symbol Multiplatine-rescue:Ferrite_Bead_Small-Device
- added J1, J5, J6: (no value), symbol Connector:Conn_01x04_Female
- added J10: (no value), symbol Connector:Conn_01x02_Male
- added J12, J13: (no value), symbol Connector_Generic:Conn_02x03_Odd_Even
- added J14: (no value), symbol Connector:USB_B_Micro
- added J2, J3: (no value), symbol Connector:Screw_Terminal_01x02
- added J4: (no value), symbol Connector:Conn_01x07_Female
- added J7: (no value), symbol Connector:AudioJack3
- added J8, J9: (no value), symbol Connector:Conn_01x03_Female
- added JP1: (no value), symbol Jumper:SolderJumper_2_Open
- added Q1, Q2: (no value), symbol Transistor_BJT:S8050
- added R1, R2, R3, R4, R5, R6, R7: (no value), symbol Device:R_Small
- added S1: (no value), symbol Multiplatine-rescue:PEC11R-4215F-S0024-dk_Encoders
- added S2: (no value), symbol Multiplatine-rescue:JS5208-dk_Navigation-Switches-Joystick
- added S3: (no value), symbol Multiplatine-rescue:NAV_SWITCH-SparkFun-Switches
- added SW1: (no value), symbol Switch:SW_Push
- added TP1, TP2, TP3: (no value), symbol Connector:TestPoint
- added U1, U3: (no value), symbol Multiplatine-rescue:MAX98357AETE+T-MAX98357AETE_T_I2S
- added U2: (no value), symbol Multiplatine-rescue:ESP32-WROVER-esp32-wrover
- added U4: (no value), symbol Regulator_Linear:AMS1117-3.3
- added U5: (no value), symbol Multiplatine-rescue:I2S-Mems-Mic-BesmerLabs
- added U6: (no value), symbol Power_Protection:USBLC6-2SC6
- added U7: (no value), symbol Interface_USB:CH340G
- added Y1: (no value), symbol Device:Crystal_GND2
Connections:
- new net: C2.1, FB1.1, J2.1 (Pin_1)
- new net: FB1.2, U3.10 (OUTN)
- new net: C1.1, FB2.1, J2.2 (Pin_2)
- new net: FB2.2, U3.9 (OUTP)
- new net: FB3.2, U1.10 (OUTN)
- new net: R1.1, TP1.1, U1.4 (SD_MODE)
- new net: FB4.2, U1.9 (OUTP)
- new net: Q2.1 (E), R6.2, U7.13 (~{DTR})
- new net: Q1.1 (E), R7.2, U7.14 (~{RTS})
- new net: R4.2, U7.2 (TXD)
- new net: R5.2, U7.3 (RXD)
- new net: C14.1, U7.7 (XI), Y1.1
- new net: C15.1, U7.8 (XO), Y1.3
- new net: Q1.2 (B), R6.1
- new net: Q2.2 (B), R7.1
- new net: C8.1, FB3.1, J3.1 (Pin_1)
- new net: C6.1, FB4.1, J3.2 (Pin_2)
- new net: D2.2 (DOUT), D3.4 (DIN)
- new net: D3.2 (DOUT), D4.4 (DIN)
- new net: D1.1 (K), R2.1
- new net +3V3: C10.1, C13.1, C16.2, C17.1, C3.1, C4.1, C5.1, C7.1, C9.1, D1.2 (A), D2.1 (VDD), D3.1 (VDD), D4.1 (VDD), J1.2 (Pin_2), J13.4 (Pin_4), J5.2 (Pin_2), J6.1 (Pin_1), J9.2 (Pin_2), R1.2, R3.2, U1.7 (VDD), U1.8 (VDD), U2.2 (3V3), U3.4 (SD_MODE), U3.7 (VDD), U3.8 (VDD), U4.2 (VO), U5.1 (3V), U7.16 (VCC), U7.4 (V3)
- new net +5V: C12.2, D5.1 (K), J4.1 (Pin_1), U4.3 (VI)
- new net +BATT: BT1.1 (+), J10.2 (Pin_2), TP2.1
- new net -BATT: BT1.2 (-), J10.1 (Pin_1), TP3.1
- new net 1WIRE: J7.T, J8.2 (Pin_2), U2.26 (IO4)
- new net BRIGHTNESS_ANALOG: J6.4 (Pin_4), U2.11 (IO26)
- new net BRIGHTNESS_DIGITAL: J6.3 (Pin_3), U2.10 (IO25)
- new net EN: C11.2, Q1.3 (C), R3.1, U2.3 (EN)
- new net GND: C1.2, C10.2, C11.1, C12.1, C13.2, C14.2, C15.2, C16.1, C17.2, C2.2, C3.2, C4.2, C5.2, C6.2, C7.2, C8.2, C9.2, D2.3 (VSS), D3.3 (VSS), D4.3 (VSS), J1.1 (Pin_1), J12.3 (Pin_3), J13.2 (Pin_2), J14.4 (ID), J14.5 (GND), J14.6 (Shield), J4.7 (Pin_7), J5.1 (Pin_1), J6.2 (Pin_2), J7.R, J7.S, J8.1 (Pin_1), J8.3 (Pin_3), J9.1 (Pin_1), JP1.2 (B), R2.2, S1.2, S1.3, S1.C (COM), U1.11 (GND), U1.15 (GND), U1.3 (GND), U2.1 (GND), U2.15 (GND), U2.38 (GND), U2.39 (GND), U3.11 (GND), U3.15 (GND), U3.3 (GND), U4.1 (GND), U5.2 (GND), U5.6 (SEL), U6.2 (GND), U7.1 (GND), Y1.2
- new net I2C_SCL: J1.4 (Pin_4), J5.3 (Pin_3), U2.19 (CMD_IO11)
- new net I2C_SDA: J1.3 (Pin_3), J5.4 (Pin_4), U2.18 (SD3_IO10)
- new net I2S_BCK: J12.5 (Pin_5), U1.16 (BCLK), U2.33 (IO21), U3.16 (BCLK), U5.3 (BCLK)
- new net I2S_DATA_IN: J13.6 (Pin_6), U2.6 (IO34), U5.4 (DOUT)
- new net I2S_DATA_OUT: U1.1 (DIN), U2.12 (IO27), U3.1 (DIN)
- new net I2S_LRCLK: J12.1 (Pin_1), U1.14 (LRCLK), U2.36 (IO22), U3.14 (LRCLK), U5.5 (LRCLK)
- new net I2S_OUTPUT_GAIN: JP1.1 (A), U1.2 (GAIN_SLOT), U3.2 (GAIN_SLOT)
- new net IO0: Q2.3 (C)
- new net NEOPIXEL: D2.4 (DIN), U2.14 (IO12)
- new net ROTARY_A: S1.A (CH_A), U2.8 (IO32_XTAL_32K_P)
- new net ROTARY_B: S1.B (CH_B), U2.9 (IO33_XTAL_32K_N)
- new net ROTARY_SWITCH: S1.1, U2.7 (IO35)
- new net RX: R4.1, U2.34 (RXD0)
- new net SPI_CS: J4.3 (Pin_3), U2.29 (IO5)
- new net SPI_MISO: J4.6 (Pin_6), U2.31 (IO19)
- new net SPI_MOSI: J4.4 (Pin_4), U2.37 (IO23)
- new net SPI_SCK: J4.5 (Pin_5), U2.30 (IO18)
- new net TX: R5.1, U2.35 (TXD0)
- new net USB_CONN_D+: J14.3 (D+), U6.6 (I/O1)
- new net USB_CONN_D-: J14.2 (D-), U6.4 (I/O2)
- new net USB_D+: U6.1 (I/O1), U7.5 (UD+)
- new net USB_D-: U6.3 (I/O2), U7.6 (UD-)
- new net VUSB: D5.2 (A), J14.1 (VBUS), U6.5 (VBUS)
- no-connect marks 0 -> 12
